File: EaglePanelizer/PGA44DIP44.brd (EAGLE design)
At the start: 58.4 x 20.3 mm, 9 parts, among them CN1 JTAG, IC1 LM2937ET-3.3/NOPB

Commit message: Update sample
Parts:
- added JP2: VCCINT, PGA44DIP44:1X01
- added LED1: TLLR4400, PGA44DIP44:LED3MM
- added R1: 1K, PGA44DIP44:0207/2V
- moved IC1 0.63 mm to (3.17, 12.1)
- moved JP1 0.63 mm to (8.26, 9.53)
Connections:
- new net N$1: LED1.K, R1.2
- net GND: now also R1.1
- net VCCINT: now also JP2.1, LED1.A
Routing:
- net N$1: track 0.00 -> 2.17 mm
- net L22: track 20.9 -> 23.0 mm
- net VCCINT: track 62.9 -> 64.8 mm
- net L3: track 19.2 -> 20.1 mm
- net L44: track 22.0 -> 22.8 mm
- net L2: track 19.2 -> 19.8 mm
- net TDI: track 36.5 -> 37.1 mm
- net TMS: track 30.0 -> 30.5 mm, vias 1 -> 0
Other:
- board text added: "IO"
- board text added: "V33"
- board text added: "VCCINT"
